Commit message: simplified URDF

File: ros/src/jonny_robot_description/urdf/jonny.urdf (robot description, URDF)
Before this commit: robot Jonny, 8 links, 7 joints
Joints:
- joint base_joint: axis 0 0 1 -> 0 1 0
- joint joint_1: axis 0 1 0 -> 0 0 1; origin xyz=0 0 0.043358 rpy=1.5708 0 0.035851 -> xyz=0 0 0.13 rpy=0 0 0
- joint joint_2: axis 0 0 1 -> 0 -1 0; origin xyz=0 0.23664 0 rpy=0 0 0 -> xyz=0 0 0.15 rpy=0 0 0
- joint joint_3: axis 0 0 -1 -> 0 1 0; limit lower=-2.0944 upper=2.0944 effort=0 velocity=0 -> lower=-2.1 upper=2.1 effort=0 velocity=0; origin xyz=0 0.26 0 rpy=0 0 0 -> xyz=0 0 0.26 rpy=0 0 0
- joint joint_4: axis 0 -1 0 -> 0 0 -1; origin xyz=0 0.1538 0 rpy=0 -0.035851 0 -> xyz=0 0 0.159 rpy=0 0 0
- joint joint_5: axis 0 0 -1 -> 0 1 0; origin xyz=0 0.1652 0 rpy=0 0 0 -> xyz=0 0 0.16 rpy=0 0 0
- joint joint_6: axis 0 -1 0 -> 0 0 -1; origin xyz=0 0.0408 0.0003 rpy=0 0 0 -> xyz=0 0 0.041 rpy=0 0 0
